File: hardware/esp-rust-board/esp-rust-board.kicad_sch (KiCad schematic)
At the start: 53 parts, among them J1 USB4105-GF-A, Q1 DMG3415U, SW1 SW_Push, SW2 SW_Push, U1 SHTC3, U2 ICM-42670-P, U3 ESP32-C3-MINI-1, U4 Rust_Board, U5 SY8088, U6 MCP73831-2-OT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

Commit message: [HW] Add kicad symbol for WM8904
Other:
- added sheet audio_codec (audio_codec.kicad_sch)
Changed lines of the file:
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@@
     (pin "2")
+  )
+  (sheet (at 119.38 109.22) (size 35.56 15.24) (fields_autoplaced)
+    (stroke (width 0.1524) (type solid) (color 0 0 0 0))
+    (fill (color 0 0 0 0.0000))
+    (property "Sheet name" "audio_codec" (id 0) (at 119.38 108.5084 0)
+      (effects (font (size 1.27 1.27)) (justify left bottom))
+    )
+    (property "Sheet file" "audio_codec.kicad_sch" (id 1) (at 119.38 125.0446 0)
+      (effects (font (size 1.27 1.27)) (justify left top))
+    )
   )
   (sheet_instances
     (path "/" (page "1"))
+    (path "/5f8e78fa-fc97-4a96-80a4-b11b892e82f2" (page "2"))
   )
   (symbol_instances
@@
       (reference "U6") (unit 1) (value "MCP73831-2-OT") (footprint "Package_TO_SOT_SMD:SOT-23-5")
     )
+    (path "/5f8e78fa-fc97-4a96-80a4-b11b892e82f2/60df69da-dd0d-4654-9e3f-9e1c8ebb8c59"
+      (reference "U?") (unit 1) (value "WM8904") (footprint "Package_DFN_QFN:QFN-32-1EP_4x4mm_P0.4mm_EP2.65x2.65mm_ThermalVias")
+    )
     (path "/00000000-0000-0000-0000-00006234eeee"
